Commit message: Update robot description to the Fusion CAD model; make sim.launch.py world-agnostic
Brings the ubot_description from the Horizon workspace, where the Inspection Robot 01
Fusion 360 model replaced the box/cylinder placeholders. Link and joint names are
unchanged, so ros2_control, Nav2, EKF, SLAM, the gz bridges and the RViz configs all
keep working.

Robot description:
- Real chassis, wheel, LD06 and camera meshes (meshes/inspection/*.stl).
- base_link is centred between the four wheels at the chassis underside; base_footprint
  on the ground. Wheel joints sit on the real axles (wheelbase 0.255 m, track 0.2264 m,
  r 32.5 mm). Collision is three boxes plus wheel cylinders, not the 52k-triangle mesh.
- camera_link is now the OAK-D Lite (4.09 deg down); new rpi_camera_link (12.54 deg down)
  with its optical frame. lidar_link sits at the real LD06 position.
- Rear wheels mimic the front ones, matching the real robot where only the front motors
  are commanded and only they have encoders.
- Wheel mu2 lowered to 0.05: a 4-wheel skid-steer must scrub its tyres to turn, and with
  equal lateral grip the wheels stall while odometry keeps integrating.
- Fixes a latent xacro bug: ubot_base, ubot_imu and ubot_ultrasonic all defined global
  properties named com_x/y/z, so base_link was silently using the IMU's centre of mass.

sim.launch.py:
- world, world_name, spawn_x/y/z/yaw are launch arguments now, defaulting to
  sonoma_occlusion and Honour's spawn pose. world_name is separate because the spawner
  addresses the world by its <world name> ('sensors'), which is not the filename.
- use_slam/use_nav2/use_rviz/headless toggles. The raceway world is expensive; running
  Gazebo plus the robot alone is usually what occlusion capture needs.
- Controller spawners get --controller-manager-timeout/--switch-timeout/--service-call-timeout.
  gz_ros2_control answers switch_controller from the simulation loop, which in a heavy
  world stalls past the 10 s default and kills the spawner with "Failed to acquire lock".

Worlds:
- sonoma_occlusion_lite.sdf: same occlusion scene, raceway terrain replaced by a ground
  plane at z=3.2. The full raceway mesh stalls machines without GPU passthrough (WSL);
  the lite world runs at real-time factor 1.0 with the robot spawned.
- apartment.sdf + models/apartment: indoor corridor world for navigation testing.

Also disables the slam_toolbox map_file_name pointing at /home/chibueze/uni-bot, which
only exists on one laptop and errored on every start.

Co-Authored-By: Claude Opus 5 <noreply@anthropic.com>

File: occlusion-sim/src/ubot/ubot_description/urdf/body/ubot_base.urdf.xacro (robot description, xacro)
@@ -1,38 +1,72 @@
 <?xml version="1.0"?>
 <robot xmlns:xacro="http://www.ros.org/wiki/xacro">
-<xacro:property name="base_width" value="0.2371" />
-<xacro:property name="base_length" value="0.41" />
-<xacro:property name="base_height" value="0.2025" />
-<xacro:property name="com_x" value="0.00489" />     <!--Center of Mass-->
-<xacro:property name="com_y" value="-0.00007433" />
-<xacro:property name="com_z" value="0.001" />
-<xacro:property name="base_mass" value="3.0" />
+<!--
+  Inspection Robot 01 chassis (exported from Fusion 360, see meshes/inspection/).
+  Frame convention (REP-105):
+    base_footprint : on the ground, centred between the four wheels
+    base_link      : centred between the four wheels, at the underside of the chassis
+                     X forward (OAK-D side), Y left, Z up
+  The chassis mesh is exported in Fusion world coordinates (mm). base_link sits at
+  Fusion point (162.38, 0, 0) mm, hence the mesh origin offset below.
+-->
+<xacro:property name="base_mesh_x" value="-0.16238" />       <!-- Fusion origin -> base_link -->
+<xacro:property name="ground_clearance" value="0.066375" />  <!-- base_link height above ground (wheel r 32.5 mm + axle 33.875 mm below chassis) -->
+<!-- Mass properties from CAD (PLA printed parts at 100% infill, aluminium motors, LCD).
+     Real robot will be heavier (battery, Pi, wiring) and lighter where printed at partial infill. -->
+<xacro:property name="base_mass" value="1.757604" />
+<xacro:property name="base_com_x" value="0.010371" />
+<xacro:property name="base_com_y" value="-0.000052" />
+<xacro:property name="base_com_z" value="0.051079" />
+<!-- Simplified collision boxes (the full mesh has ~52k triangles, too heavy for physics) -->
+<xacro:property name="body_length" value="0.357" />
+<xacro:property name="body_width" value="0.220" />
+<xacro:property name="body_height" value="0.173" />
+<xacro:property name="body_x" value="0.00088" />
+<xacro:property name="mast_length" value="0.102" />
+<xacro:property name="mast_width" value="0.066" />
+<xacro:property name="mast_height" value="0.107" />
+<xacro:property name="mast_x" value="0.0610" />
+<xacro:property name="mast_z" value="0.2265" />
+<!-- Motors and holders hang below the chassis (z -0.048 .. 0), i.e. 18 mm above the ground. -->
+<xacro:property name="under_length" value="0.336" />
+<xacro:property name="under_width" value="0.232" />
+<xacro:property name="under_height" value="0.048" />
+<xacro:property name="under_z" value="-0.024" />
 <xacro:macro name="ubot_base" params="prefix">
-    <link name="base_footprint"/>
+    <link name="${prefix}base_footprint"/>
     <link name="${prefix}base_link">
         <visual>
-            <!-- <geometry>
-                <mesh filename="file://$(find ubot_description)/meshes/latest.stl" scale="1 1 1"/>
-            </geometry> -->
+            <origin xyz="${base_mesh_x} 0 0" rpy="0 0 0"/>
             <geometry>
-                <box size="${base_length} ${base_width} ${base_height}"/>
+                <mesh filename="file://$(find ubot_description)/meshes/inspection/base.stl" scale="0.001 0.001 0.001"/>
             </geometry>
-            <origin xyz="0 0 ${base_height/2}" rpy="0 0 0"/>
-            <material name="dark_gray">
-                <color rgba="0.2 0.2 0.2 0.5"/>
+            <material name="chassis_gray">
+                <color rgba="0.75 0.75 0.75 1"/>
             </material>
         </visual>
         <collision>
+            <origin xyz="${body_x} 0 ${body_height/2}" rpy="0 0 0"/>
             <geometry>
-                <box size="${base_length - 0.01} ${base_width - 0.01} ${base_height - 0.01}"/>
+                <box size="${body_length} ${body_width} ${body_height}"/>
             </geometry>
-            <origin xyz="0 0 ${base_height/2}" rpy="0 0 0"/>
+        </collision>
+        <collision>
+            <origin xyz="${mast_x} 0 ${mast_z}" rpy="0 0 0"/>
+            <geometry>
+                <box size="${mast_length} ${mast_width} ${mast_height}"/>
+            </geometry>
+        </collision>
+        <collision>
+            <origin xyz="0 0 ${under_z}" rpy="0 0 0"/>
+            <geometry>
+                <box size="${under_length} ${under_width} ${under_height}"/>
+            </geometry>
         </collision>
         <inertial>
-            <origin xyz="${com_x} ${com_y} ${com_z}" rpy="0 0 0"/>
+            <origin xyz="${base_com_x} ${base_com_y} ${base_com_z}" rpy="0 0 0"/>
             <mass value="${base_mass}"/>
-            <inertia ixx="${(1/12) * base_mass * ((base_width * base_width) + (base_height * base_height))}"  ixy="0.0"  ixz="0.0"
-                     iyy="${(1/12) * base_mass * ((base_length * base_length) + (base_height * base_height))}"  iyz="0.0"
-                     izz="${(1/12) * base_mass * ((base_length * base_length) + (base_width * base_width))}"/>
+            <inertia ixx="0.019834" ixy="-0.000003" ixz="-0.001273"
+                     iyy="0.034307" iyz="0.000005"
+                     izz="0.033227"/>
         </inertial>
     </link>
@@ -40,7 +74,7 @@
         <visual>
             <material>
-                <ambient>0.5 0.5 0.5 0.5</ambient>
-                <diffuse>0.5 0.5 0.5 0.5</diffuse>
-                <specular>0.2 0.2 0.2 0.5</specular>
+                <ambient>0.6 0.6 0.6 1</ambient>
+                <diffuse>0.75 0.75 0.75 1</diffuse>
+                <specular>0.2 0.2 0.2 1</specular>
             </material>
         </visual>
@@ -49,5 +83,5 @@
         <parent link="${prefix}base_footprint"/>
         <child link="${prefix}base_link"/>
-        <origin xyz="0 0 ${wheel_radius - wheel_zoff}" rpy="0 0 0"/>
+        <origin xyz="0 0 ${ground_clearance}" rpy="0 0 0"/>
   </joint>
 </xacro:macro>

File: occlusion-sim/src/ubot/ubot_description/urdf/body/ubot_robot.urdf.xacro (robot description, xacro)
@@ -7,6 +7,8 @@
     <xacro:include filename="$(find ubot_description)/urdf/body/ubot_base.urdf.xacro"/>
     <xacro:include filename="$(find ubot_description)/urdf/sensors/ubot_lidar.urdf.xacro"/>
-    <xacro:include filename="$(find ubot_description)/urdf/sensors/ubot_ultrasonic.urdf.xacro"/>
+    <!-- Ultrasonics are not part of the Inspection Robot 01 body; re-enable here and below if fitted. -->
+    <!-- <xacro:include filename="$(find ubot_description)/urdf/sensors/ubot_ultrasonic.urdf.xacro"/> -->
     <xacro:include filename="$(find ubot_description)/urdf/sensors/ubot_camera.urdf.xacro"/>
+    <xacro:include filename="$(find ubot_description)/urdf/sensors/ubot_rpi_camera.urdf.xacro"/>
     <xacro:include filename="$(find ubot_description)/urdf/sensors/ubot_imu.urdf.xacro"/>
     <xacro:include filename="$(find ubot_description)/urdf/body/ubot_wheel.urdf.xacro"/>
@@ -23,7 +25,9 @@
     <xacro:ubot_lidar
     prefix="$(arg prefix)" />
-    <xacro:ubot_ultrasonic
+    <!-- <xacro:ubot_ultrasonic
+    prefix="$(arg prefix)" /> -->
+    <xacro:ubot_camera
     prefix="$(arg prefix)" />
-    <xacro:ubot_camera
+    <xacro:ubot_rpi_camera
     prefix="$(arg prefix)" />
     <xacro:ubot_imu

File: occlusion-sim/src/ubot/ubot_description/urdf/body/ubot_wheel.urdf.xacro (robot description, xacro)
@@ -1,25 +1,30 @@
 <?xml version="1.0"?>
 <robot xmlns:xacro="http://www.ros.org/wiki/xacro">
-  <xacro:property name="wheel_radius" value="0.033" />
-  <xacro:property name="wheel_separation" value="0.264204" />  <!-- 2 * wheel_yoff = 2 * (base_width/2 + motor_cylinder_length) -->
+  <!-- Geometry from CAD (Inspection Robot 01). Joint origins sit exactly on each motor axle. -->
+  <xacro:property name="wheel_radius" value="0.0325" />
   <xacro:property name="wheel_width" value="0.0264" />
-  <xacro:property name="wheel_mass" value="0.4" />
-  <xacro:property name="back_to_front_wheel" value="0.3043" />
-  <xacro:property name="back_to_rear_wheel" value="0.056536" />
-  <xacro:property name="wheel_xoff1" value="${back_to_front_wheel - base_length/2}" />
-  <xacro:property name="wheel_xoff2" value="${base_length/2 - back_to_rear_wheel}" />
-  <xacro:property name="motor_cylinder_length" value="0.013552" />
-  <xacro:property name="wheel_yoff" value="${base_width/2 + motor_cylinder_length}" />
-  <xacro:property name="wheel_zoff" value="0.0188" /> <!--0.018805-->
-  <xacro:macro name="ubot_wheel" params="prefix">
-    <link name="${prefix}front_left_wheel_link">
+  <xacro:property name="wheel_xoff" value="0.1275" />       <!-- half wheelbase (0.255 m axle to axle) -->
+  <xacro:property name="wheel_yoff" value="0.1132" />       <!-- half track, wheel centre plane -->
+  <xacro:property name="wheel_zoff" value="-0.033875" />    <!-- axle below base_link -->
+  <xacro:property name="wheel_separation" value="${2*wheel_yoff}" />  <!-- geometric 0.2264 m -->
+  <xacro:property name="wheel_mass" value="0.044215" />
+  <xacro:property name="wheel_ixx" value="0.000018" />
+  <xacro:property name="wheel_iyy" value="0.000032" />      <!-- about the axle -->
+  <xacro:property name="wheel_izz" value="0.000018" />
+  <!-- Wheel meshes are in Fusion world coordinates (mm): mesh_x/mesh_y is the wheel
+       centre in that frame, so the visual origin is its negative. -->
+  <!--
+    mimics: name of the joint this wheel's joint follows, or "" for a driven/sensed wheel.
+    The real robot commands only the FRONT motors; the ESP32 mirrors each front command to
+    the rear motor on the same side, and only the front wheels carry encoders. Declaring the
+    rear joints as URDF mimic joints reproduces that exactly: gz_ros2_control copies the
+    front command onto the rear joint, and the rear joints expose no command interface.
+  -->
+  <xacro:macro name="ubot_single_wheel" params="prefix name x_sign y_sign mesh mesh_x mesh_y mimics:=''">
+    <link name="${prefix}${name}_wheel_link">
       <visual>
-        <!-- <geometry>
-            <mesh filename="package://ubot_description/meshes/wheel.stl" scale="0.001 0.001 0.001"/>
-        </geometry> -->
-        <!-- <origin xyz="0 0 0" rpy="0 0 ${-pi/2}"/> -->
-        <origin xyz="0 0 0" rpy="${pi/2} 0 0"/>
+        <origin xyz="${-mesh_x} ${-mesh_y} ${-wheel_zoff}" rpy="0 0 0"/>
         <geometry>
-          <cylinder radius="${wheel_radius}" length="${wheel_width}"/>
+          <mesh filename="file://$(find ubot_description)/meshes/inspection/${mesh}.stl" scale="0.001 0.001 0.001"/>
         </geometry>
         <material name="dark_gray">
@@ -36,122 +41,22 @@
         <origin xyz="0 0 0" rpy="0 0 0"/>
         <mass value="${wheel_mass}"/>
-        <inertia
-          ixx="${(wheel_mass/12.0) * (3*wheel_radius*wheel_radius + wheel_width*wheel_width)}" ixy="0" ixz="0"
-          iyy="${(wheel_mass/2.0) * (wheel_radius*wheel_radius)}" iyz="0"
-          izz="${(wheel_mass/12.0) * (3*wheel_radius*wheel_radius + wheel_width*wheel_width)}"/>
+        <inertia ixx="${wheel_ixx}" ixy="0" ixz="0" iyy="${wheel_iyy}" iyz="0" izz="${wheel_izz}"/>
       </inertial>
     </link>
-    <joint name="${prefix}front_left_wheel_joint" type="continuous">
+    <joint name="${prefix}${name}_wheel_joint" type="continuous">
       <axis xyz="0 1 0"/>
       <parent link="${prefix}base_link"/>
-      <child link="${prefix}front_left_wheel_link"/>
-      <!-- <origin xyz="${x_reflect*(wheel_xoff) } ${y_reflect*(wheel_yoff)} ${-wheel_zoff}" rpy="0 0 0"/> -->
-      <origin xyz="${wheel_xoff1} ${wheel_yoff} ${wheel_zoff}" rpy="0 0 0"/>
-    </joint>
-    <link name="${prefix}front_right_wheel_link">
-      <visual>
-        <!-- <geometry>
-            <mesh filename="package://ubot_description/meshes/wheel.stl" scale="0.001 0.001 0.001"/>
-        </geometry>
-        <origin xyz="0 0 0" rpy="0 0 ${pi/2}"/> -->
-        <origin xyz="0 0 0" rpy="${pi/2} 0 0"/>
-        <geometry>
-          <cylinder radius="${wheel_radius}" length="${wheel_width}"/>
-        </geometry>
-        <material name="dark_gray">
-          <color rgba="0.2 0.2 0.2 1"/>
-        </material>
-      </visual>
-      <collision>
-        <origin xyz="0 0 0" rpy="${pi/2} 0 0"/>
-        <geometry>
-          <cylinder radius="${wheel_radius}" length="${wheel_width}"/>
-        </geometry>
-      </collision>
-      <inertial>
-        <origin xyz="0 0 0" rpy="0 0 0"/>
-        <mass value="${wheel_mass}"/>
-        <inertia
-          ixx="${(wheel_mass/12.0) * (3*wheel_radius*wheel_radius + wheel_width*wheel_width)}" ixy="0" ixz="0"
-          iyy="${(wheel_mass/2.0) * (wheel_radius*wheel_radius)}" iyz="0"
-          izz="${(wheel_mass/12.0) * (3*wheel_radius*wheel_radius + wheel_width*wheel_width)}"/>
-      </inertial>
-    </link>
-    <joint name="${prefix}front_right_wheel_joint" type="continuous">
-      <axis xyz="0 1 0"/>
-      <parent link="${prefix}base_link"/>
-      <child link="${prefix}front_right_wheel_link"/>
-      <origin xyz="${wheel_xoff1} ${-wheel_yoff} ${wheel_zoff}" rpy="0 0 0"/>
-    </joint>
-    <link name="${prefix}rear_left_wheel_link">
-      <visual>
-        <!-- <geometry>
-            <mesh filename="package://ubot_description/meshes/wheel.stl" scale="0.001 0.001 0.001"/>
-        </geometry>
-        <origin xyz="0 0 0" rpy="0 0 ${pi/2}"/> -->
-        <origin xyz="0 0 0" rpy="${pi/2} 0 0"/>
-        <geometry>
-          <cylinder radius="${wheel_radius}" length="${wheel_width}"/>
-        </geometry>
-        <material name="dark_gray">
-          <color rgba="0.2 0.2 0.2 1"/>
-        </material>
-      </visual>
-      <collision>
-        <origin xyz="0 0 0" rpy="${pi/2} 0 0"/>
-        <geometry>
-          <cylinder radius="${wheel_radius}" length="${wheel_width}"/>
-        </geometry>
-      </collision>
-      <inertial>
-        <origin xyz="0 0 0" rpy="0 0 0"/>
-        <mass value="${wheel_mass}"/>
-        <inertia
-          ixx="${(wheel_mass/12.0) * (3*wheel_radius*wheel_radius + wheel_width*wheel_width)}" ixy="0" ixz="0"
-          iyy="${(wheel_mass/2.0) * (wheel_radius*wheel_radius)}" iyz="0"
-          izz="${(wheel_mass/12.0) * (3*wheel_radius*wheel_radius + wheel_width*wheel_width)}"/>
-      </inertial>
-    </link>
-    <joint name="${prefix}rear_left_wheel_joint" type="continuous">
-      <parent link="${prefix}base_link"/>
-      <child link="${prefix}rear_left_wheel_link"/>
-      <origin xyz="${-wheel_xoff2} ${wheel_yoff} ${wheel_zoff}" rpy="0 0 0"/>
-      <axis xyz="0 1 0"/>
-    </joint>
-    <link name="${prefix}rear_right_wheel_link">
-      <visual>
-        <!-- <geometry>
-            <mesh filename="package://ubot_description/meshes/wheel.stl" scale="0.001 0.001 0.001"/>
-        </geometry>
-        <origin xyz="0 0 0" rpy="0 0 ${pi/2}"/> -->
-        <origin xyz="0 0 0" rpy="${pi/2} 0 0"/>
-        <geometry>
-          <cylinder radius="${wheel_radius}" length="${wheel_width}"/>
-        </geometry>
-        <material name="dark_gray">
-          <color rgba="0.2 0.2 0.2 1"/>
-        </material>
-      </visual>
-      <collision>
-        <origin xyz="0 0 0" rpy="${pi/2} 0 0"/>
-        <geometry>
-          <cylinder radius="${wheel_radius}" length="${wheel_width}"/>
-        </geometry>
-      </collision>
-      <inertial>
-        <origin xyz="0 0 0" rpy="0 0 0"/>
-        <mass value="${wheel_mass}"/>
-        <inertia
-          ixx="${(wheel_mass/12.0) * (3*wheel_radius*wheel_radius + wheel_width*wheel_width)}" ixy="0" ixz="0"
-          iyy="${(wheel_mass/2.0) * (wheel_radius*wheel_radius)}" iyz="0"
-          izz="${(wheel_mass/12.0) * (3*wheel_radius*wheel_radius + wheel_width*wheel_width)}"/>
-      </inertial>
-    </link>
-    <joint name="${prefix}rear_right_wheel_joint" type="continuous">
-      <parent link="${prefix}base_link"/>
-      <child link="${prefix}rear_right_wheel_link"/>
-      <origin xyz="${-wheel_xoff2} ${-wheel_yoff} ${wheel_zoff}" rpy="0 0 0"/>
-      <axis xyz="0 1 0"/>
+      <child link="${prefix}${name}_wheel_link"/>
+      <origin xyz="${x_sign*wheel_xoff} ${y_sign*wheel_yoff} ${wheel_zoff}" rpy="0 0 0"/>
+      <xacro:unless value="${mimics == ''}">
+        <mimic joint="${prefix}${mimics}" multiplier="1.0" offset="0.0"/>
+      </xacro:unless>
     </joint>
   </xacro:macro>
+  <xacro:macro name="ubot_wheel" params="prefix">
+    <xacro:ubot_single_wheel prefix="${prefix}" name="front_left"  x_sign="1"  y_sign="1"  mesh="wheel_front_left"  mesh_x="0.28988" mesh_y="0.1132"/>
+    <xacro:ubot_single_wheel prefix="${prefix}" name="front_right" x_sign="1"  y_sign="-1" mesh="wheel_front_right" mesh_x="0.28988" mesh_y="-0.1132"/>
+    <xacro:ubot_single_wheel prefix="${prefix}" name="rear_left"   x_sign="-1" y_sign="1"  mesh="wheel_rear_left"   mesh_x="0.03488" mesh_y="0.1132"  mimics="front_left_wheel_joint"/>
+    <xacro:ubot_single_wheel prefix="${prefix}" name="rear_right"  x_sign="-1" y_sign="-1" mesh="wheel_rear_right"  mesh_x="0.03488" mesh_y="-0.1132" mimics="front_right_wheel_joint"/>
+  </xacro:macro>
 </robot>

File: occlusion-sim/src/ubot/ubot_description/urdf/gazebo/ubot_gazebo.urdf.xacro (robot description, xacro)
@@ -156,8 +156,16 @@
             </sensor>
         </gazebo>
+        <!--
+          Skid-steer friction.
+          mu1 acts along fdir1 (the rolling direction, +X) and mu2 across it (sideways).
+          A 4-wheel skid-steer can only turn by scrubbing its tyres sideways, so mu2 MUST
+          be low. With mu1 = mu2 = 1.1 the robot is effectively bolted to the floor: the
+          wheels stall while the odometry keeps integrating, so the robot spins in RViz
+          but not in Gazebo.
+        -->
         <xacro:macro name="wheel_gazebo" params="wheel_name">
             <gazebo reference="${prefix}${wheel_name}_link">
-                <mu1>1.1</mu1>
-                <mu2>1.1</mu2>
+                <mu1>1.0</mu1>
+                <mu2>0.50</mu2>
                 <kp>1000000.0</kp>
                 <kd>10.0</kd>

File: occlusion-sim/src/ubot/ubot_description/urdf/ros2_control/ubot_ros2_control.xacro (robot description, xacro)
@@ -69,7 +69,4 @@
       -->
       <joint name="${prefix}rear_left_wheel_joint">
-        <xacro:if value="${use_gazebo}">
-          <command_interface name="velocity"/>
-        </xacro:if>
         <state_interface name="position"/>
         <state_interface name="velocity"/>
@@ -77,7 +74,4 @@
       <!-- Rear right — same as rear left -->
       <joint name="${prefix}rear_right_wheel_joint">
-        <xacro:if value="${use_gazebo}">
-          <command_interface name="velocity"/>
-        </xacro:if>
         <state_interface name="position"/>
         <state_interface name="velocity"/>
