Commit message: Update robot description to the Fusion CAD model; make sim.launch.py world-agnostic
Brings the ubot_description from the Horizon workspace, where the Inspection Robot 01
Fusion 360 model replaced the box/cylinder placeholders. Link and joint names are
unchanged, so ros2_control, Nav2, EKF, SLAM, the gz bridges and the RViz configs all
keep working.

Robot description:
- Real chassis, wheel, LD06 and camera meshes (meshes/inspection/*.stl).
- base_link is centred between the four wheels at the chassis underside; base_footprint
  on the ground. Wheel joints sit on the real axles (wheelbase 0.255 m, track 0.2264 m,
  r 32.5 mm). Collision is three boxes plus wheel cylinders, not the 52k-triangle mesh.
- camera_link is now the OAK-D Lite (4.09 deg down); new rpi_camera_link (12.54 deg down)
  with its optical frame. lidar_link sits at the real LD06 position.
- Rear wheels mimic the front ones, matching the real robot where only the front motors
  are commanded and only they have encoders.
- Wheel mu2 lowered to 0.05: a 4-wheel skid-steer must scrub its tyres to turn, and with
  equal lateral grip the wheels stall while odometry keeps integrating.
- Fixes a latent xacro bug: ubot_base, ubot_imu and ubot_ultrasonic all defined global
  properties named com_x/y/z, so base_link was silently using the IMU's centre of mass.

sim.launch.py:
- world, world_name, spawn_x/y/z/yaw are launch arguments now, defaulting to
  sonoma_occlusion and Honour's spawn pose. world_name is separate because the spawner
  addresses the world by its <world name> ('sensors'), which is not the filename.
- use_slam/use_nav2/use_rviz/headless toggles. The raceway world is expensive; running
  Gazebo plus the robot alone is usually what occlusion capture needs.
- Controller spawners get --controller-manager-timeout/--switch-timeout/--service-call-timeout.
  gz_ros2_control answers switch_controller from the simulation loop, which in a heavy
  world stalls past the 10 s default and kills the spawner with "Failed to acquire lock".

Worlds:
- sonoma_occlusion_lite.sdf: same occlusion scene, raceway terrain replaced by a ground
  plane at z=3.2. The full raceway mesh stalls machines without GPU passthrough (WSL);
  the lite world runs at real-time factor 1.0 with the robot spawned.
- apartment.sdf + models/apartment: indoor corridor world for navigation testing.

Also disables the slam_toolbox map_file_name pointing at /home/chibueze/uni-bot, which
only exists on one laptop and errored on every start.

Co-Authored-By: Claude Opus 5 <noreply@anthropic.com>

File: occlusion-sim/src/ubot/ubot_description/urdf/sensors/ubot_camera.urdf.xacro (robot description, xacro)
@@ -1,53 +1,39 @@
 <?xml version="1.0"?>
 <robot xmlns:xacro="http://www.ros.org/wiki/xacro">
-  <xacro:property name="M_PI" value="3.1415926535897931" />
-  <!-- Camera Physical Properties -->
-  <xacro:property name="camera_mass" value="0.072" />  <!-- Intel RealSense D435 ~72 g -->
-  <xacro:property name="camera_width" value="0.090" />  <!-- Typical depth camera length -->
-  <xacro:property name="camera_length" value="0.025" />
-  <xacro:property name="camera_height" value="0.025" />
-  <!-- Center of Mass -->
-  <xacro:property name="com_x" value="0.0" />
-  <xacro:property name="com_y" value="0.0" />
-  <xacro:property name="com_z" value="0.0" />
-  <!-- Camera Mounting Position (relative to base_link) -->
-  <xacro:property name="camera_x" value="${base_length/2}" />
+  <!--
+    Luxonis OAK-D Lite depth camera in the front CamCase.
+    camera_link sits at the centre of the RGB lens on the front face, X pointing out of
+    the lens. The CamCase tilts the camera 4.09 deg downward (camera_pitch).
+    Mesh: simplified 91 x 28 x 17.5 mm body with the three lenses, in Fusion world coords.
+  -->
+  <xacro:property name="camera_mass" value="0.061" />    <!-- OAK-D Lite datasheet -->
+  <xacro:property name="camera_width" value="0.091" />
+  <xacro:property name="camera_length" value="0.0175" />  <!-- depth, along X -->
+  <xacro:property name="camera_height" value="0.028" />
+  <xacro:property name="camera_x" value="0.167769" />
   <xacro:property name="camera_y" value="0.0" />
-  <xacro:property name="camera_z" value="0.162618" />
+  <xacro:property name="camera_z" value="0.085654" />
+  <xacro:property name="camera_pitch" value="0.0714" />   <!-- rad, positive = looking down -->
   <xacro:macro name="ubot_camera" params="prefix">
-    <!--CAMERA_LINK (Main camera body)-->
+    <!--CAMERA_LINK (OAK-D Lite body)-->
     <link name="${prefix}camera_link">
       <visual>
+        <!-- inverse of the joint transform, so the world-frame mesh lands in place -->
+        <origin xyz="-0.323197 0 -0.108988" rpy="0 ${-camera_pitch} 0"/>
         <geometry>
-            <box size="${camera_length} ${camera_width} ${camera_height}"/>
-        </geometry>
-        <origin xyz="${-camera_length/2} 0 0" rpy="0 0 0"/>
-        <material name="camera_white">
-          <color rgba="0.9 0.9 0.9 1"/>
-        </material>
-      </visual>
-      <!-- <visual>
-        <origin xyz="0 0 0" rpy="${pi/2} 0 ${pi/2}"/>
-        <geometry>
-          <mesh filename="file://$(find ubot_description)/meshes/camera.stl" scale="0.001 0.001 0.001"/>
+          <mesh filename="file://$(find ubot_description)/meshes/inspection/oakd_lite.stl" scale="0.001 0.001 0.001"/>
         </geometry>
         <material name="camera_black">
           <color rgba="0.1 0.1 0.1 1"/>
         </material>
-      </visual> -->
-      <collision>
-        <geometry>
-            <box size="${camera_length} ${camera_width} ${camera_height}"/>
-        </geometry>
+      </visual>
+      <!-- No collision shape: the OAK-D sits inside the chassis collision box, so one here
+           would be unreachable. Add one if the camera is ever mounted proud of the body. -->
+      <inertial>
         <origin xyz="${-camera_length/2} 0 0" rpy="0 0 0"/>
-      </collision>
-      <inertial>
-        <origin xyz="${com_x} ${com_y} ${com_z}" rpy="0 0 0"/>
         <mass value="${camera_mass}"/>
-        <inertia ixx="${(1/12) * camera_mass * ((camera_width * camera_width) + (camera_height * camera_height))}"
-                 ixy="0.0"  ixz="0.0"
-                 iyy="${(1/12) * camera_mass * ((camera_length * camera_length) + (camera_height * camera_height))}"
-                 iyz="0.0"
-                 izz="${(1/12) * camera_mass * ((camera_length * camera_length) + (camera_width * camera_width))}"/>
+        <inertia ixx="0.000046" ixy="0.0" ixz="0.0"
+                 iyy="0.000006" iyz="0.0"
+                 izz="0.000044"/>
       </inertial>
     </link>
@@ -55,5 +41,5 @@
       <parent link="${prefix}base_link"/>
       <child link="${prefix}camera_link"/>
-      <origin xyz="${camera_x} ${camera_y} ${camera_z}" rpy="0 0 0"/>
+      <origin xyz="${camera_x} ${camera_y} ${camera_z}" rpy="0 ${camera_pitch} 0"/>
     </joint>
     <!-- CAMERA_DEPTH_FRAME (Optical frame for depth)
@@ -83,42 +69,2 @@
   </xacro:macro>
 </robot>
-<!-- <?xml version="1.0"?>
-<robot xmlns:xacro="http://www.ros.org/wiki/xacro">
-  <xacro:property name="M_PI" value="3.1415926535897931" />
-  <xacro:property name="camera_mass" value="0.10321" />
-  <xacro:property name="camera_length" value="0.035" />
-  <xacro:property name="camera_width" value="0.035" />
-  <xacro:property name="camera_height" value="0.035" />
-  <xacro:property name="com_x" value="-0.000082" />     Center of Mass
-  <xacro:property name="com_y" value="-0.000041" />
-  <xacro:property name="com_z" value="0.010541" />
-  <xacro:property name="stand_height" value="${camera_height}" />
-  <xacro:property name="camera_x" value="0.143122" />
-  <xacro:property name="camera_y" value="0.0" />
-  <xacro:property name="camera_z" value="0.162618" />
-  <xacro:macro name="ubot_camera" params="prefix">
-    <link name="camera_link">
-      <visual>
-        <origin xyz="0 0 0" rpy="${pi/2} 0 ${pi/2}"/>
-        <geometry>
-            <mesh filename="file://$(find ubot_description)/meshes/camera.stl" scale="0.001 0.001 0.001"/>
-        </geometry>
-        <material name="white">
-          <color rgba="1 1 1 1"/>
-        </material>
-      </visual>
-      <inertial>
-          <origin xyz="${com_x} ${com_y} ${com_z}" rpy="0 0 0"/>
-          <mass value="${camera_mass*1.25}"/>
-          <inertia ixx="${(1/12) * camera_mass * ((camera_width * camera_width) + (camera_height * camera_height))}"  ixy="0.0"  ixz="0.0"
-                    iyy="${(1/12) * camera_mass * ((camera_length * camera_length) + (camera_height * camera_height))}"  iyz="0.0"
-                    izz="${(1/12) * camera_mass * ((camera_length * camera_length) + (camera_width * camera_width))}"/>
-      </inertial>
-    </link>
-    <joint name="${prefix}camera_joint" type="fixed">
-      <parent link="base_link"/>
-      <child link="camera_link"/>
-      <origin xyz="${camera_x} ${camera_y} ${camera_z}" rpy="0 0 0"/>
-    </joint>
-  </xacro:macro>
-</robot> -->

File: occlusion-sim/src/ubot/ubot_description/urdf/sensors/ubot_imu.urdf.xacro (robot description, xacro)
@@ -6,10 +6,12 @@
   <xacro:property name="imu_width" value="0.0155" />
   <xacro:property name="imu_height" value="0.015" />
-  <xacro:property name="com_x" value="-0.000082" />     <!--Center of Mass-->
-  <xacro:property name="com_y" value="-0.000041" />
-  <xacro:property name="com_z" value="0.010541" />
-  <xacro:property name="stand_height" value="${imu_height}" />
-  <xacro:property name="imu_x" value="${-(base_length/2 - 0.115)}" />
-  <xacro:property name="imu_y" value="${-(0.165 - base_width/2)}" />
+  <xacro:property name="imu_com_x" value="-0.000082" />     <!--Center of Mass-->
+  <xacro:property name="imu_com_y" value="-0.000041" />
+  <xacro:property name="imu_com_z" value="0.010541" />
+  <!-- TODO: measure on the Inspection Robot body. These are the values from the old
+       box model (-(0.41/2 - 0.115), -(0.165 - 0.2371/2), 0.18), kept so the IMU frame
+       does not move; z = 0.18 is above the new chassis roof at this x. -->
+  <xacro:property name="imu_x" value="-0.09" />
+  <xacro:property name="imu_y" value="-0.04645" />
   <xacro:property name="imu_z" value="0.18" />
   <xacro:macro name="ubot_imu" params="prefix">
@@ -28,5 +30,5 @@
       </visual>
       <inertial>
-          <origin xyz="${com_x} ${com_y} ${com_z}" rpy="0 0 0"/>
+          <origin xyz="${imu_com_x} ${imu_com_y} ${imu_com_z}" rpy="0 0 0"/>
           <mass value="${imu_mass}"/>
           <inertia ixx="${(1/12) * imu_mass * ((imu_width * imu_width) + (imu_height * imu_height))}"  ixy="0.0"  ixz="0.0"

File: occlusion-sim/src/ubot/ubot_description/urdf/sensors/ubot_lidar.urdf.xacro (robot description, xacro)
@@ -1,43 +1,49 @@
 <?xml version="1.0"?>
 <robot xmlns:xacro="http://www.ros.org/wiki/xacro">
-  <xacro:property name="M_PI" value="3.1415926535897931" />
-  <xacro:property name="lidar_mass" value="0.170" />  <!-- RPLIDAR A1/A2 ~170 g -->
-  <xacro:property name="lidar_length" value="0.035" />
-  <xacro:property name="lidar_width" value="0.035" />
-  <xacro:property name="lidar_height" value="0.02580" />
-  <xacro:property name="com_x" value="-0.000082" />     <!--Center of Mass-->
-  <xacro:property name="com_y" value="-0.000041" />
-  <xacro:property name="com_z" value="0.010541" />
-  <xacro:property name="stand_height" value="${lidar_height}" />
-  <xacro:property name="lidar_x" value="-0.14250" />
+  <!--
+    Orbbec/Oradar MS200 dToF lidar on top of the mast.
+    The CAD models an LDROBOT LD06 (the previous sensor); the robot now runs an MS200
+    (real_robot.launch.py: device_model MS200 on /dev/ttyACM0). The two are nearly the
+    same envelope - LD06 38.6 x 38.6 x 34.8 mm, MS200 37.7 x 37.5 x 33.0 mm - so the
+    mount is unchanged and the sensor is drawn as a correctly sized primitive rather
+    than the wrong sensor's mesh.
+    lidar_link is placed at the mid-height of the sensor body. TODO: measure the real
+    scan-plane height above the mast and set lidar_scan_z; being a centimetre out in Z
+    tilts nothing but does bias obstacle heights slightly.
+  -->
+  <xacro:property name="lidar_length" value="0.0377" />   <!-- X -->
+  <xacro:property name="lidar_width"  value="0.0375" />   <!-- Y -->
+  <xacro:property name="lidar_height" value="0.0330" />   <!-- Z -->
+  <xacro:property name="lidar_mass"   value="0.0428" />   <!-- approximate, not from datasheet -->
+  <!-- Mount: top face of the mast, from CAD (base_link frame) -->
+  <xacro:property name="lidar_mount_z" value="0.2798" />
+  <xacro:property name="lidar_x" value="0.030584" />
   <xacro:property name="lidar_y" value="0.0" />
-  <xacro:property name="lidar_z" value="${base_height + lidar_height/2}" />
+  <xacro:property name="lidar_scan_z" value="${lidar_mount_z + lidar_height/2}" />
   <xacro:macro name="ubot_lidar" params="prefix">
     <link name="${prefix}lidar_link">
       <visual>
-        <origin xyz="0 0 ${-lidar_height/4}" rpy="0 0 0"/>
-        <!-- <geometry>
-            <mesh filename="file://$(find ubot_description)/meshes/lidar.stl" scale="0.001 0.001 0.001"/>
-        </geometry> -->
+        <origin xyz="0 0 0" rpy="0 0 0"/>
         <geometry>
-          <cylinder radius="${lidar_width/2}" length="${lidar_height/2}"/>
+          <box size="${lidar_length} ${lidar_width} ${lidar_height}"/>
         </geometry>
         <material name="black">
-          <color rgba="0 0 0 0.5"/>
+          <color rgba="0.05 0.05 0.05 1"/>
         </material>
       </visual>
       <collision>
-        <origin xyz="0 0 ${-lidar_height/4}" rpy="0 0 0"/>
+        <origin xyz="0 0 0" rpy="0 0 0"/>
         <geometry>
-          <cylinder radius="${lidar_width/2}" length="${lidar_height/2}"/>
+          <box size="${lidar_length} ${lidar_width} ${lidar_height}"/>
         </geometry>
       </collision>
       <inertial>
-          <origin xyz="${com_x} ${com_y} ${com_z}" rpy="0 0 0"/>
-          <mass value="${lidar_mass}"/>
-          <!-- Cylinder inertia: r = lidar_width/2, h = lidar_height -->
-          <inertia ixx="${(1/12) * lidar_mass * (3*(lidar_width/2)*(lidar_width/2) + lidar_height*lidar_height)}"  ixy="0.0"  ixz="0.0"
-                    iyy="${(1/12) * lidar_mass * (3*(lidar_width/2)*(lidar_width/2) + lidar_height*lidar_height)}"  iyz="0.0"
-                    izz="${(1/2) * lidar_mass * (lidar_width/2)*(lidar_width/2)}"/>
+        <origin xyz="0 0 0" rpy="0 0 0"/>
+        <mass value="${lidar_mass}"/>
+        <inertia ixx="${(1/12) * lidar_mass * (lidar_width*lidar_width + lidar_height*lidar_height)}"
+                 ixy="0.0" ixz="0.0"
+                 iyy="${(1/12) * lidar_mass * (lidar_length*lidar_length + lidar_height*lidar_height)}"
+                 iyz="0.0"
+                 izz="${(1/12) * lidar_mass * (lidar_length*lidar_length + lidar_width*lidar_width)}"/>
       </inertial>
     </link>
@@ -45,5 +51,5 @@
       <parent link="${prefix}base_link"/>
       <child link="${prefix}lidar_link"/>
-      <origin xyz="${lidar_x} ${lidar_y} ${lidar_z}" rpy="0 0 0"/>
+      <origin xyz="${lidar_x} ${lidar_y} ${lidar_scan_z}" rpy="0 0 0"/>
     </joint>
   </xacro:macro>
