Commit message: Add sensor_profile:=fast to trade sensor fidelity for simulation speed
Rendering the depth camera and lidar is what limits simulation speed. In the full
Sonoma Raceway world the nominal sensors run at about RTF 0.2 on a machine without
GPU passthrough: /scan arrives at ~2 Hz instead of its configured 10 Hz, so
everything is 5x slow motion.

  full (default) lidar 720 @10 Hz, camera 640x480 @30 Hz, imu @100 Hz
  fast           lidar 360 @5 Hz,  camera 320x240 @10 Hz, imu @50 Hz

  ros2 launch ubot_bringup sim.launch.py sensor_profile:=fast

Verified both profiles expand to the intended values.

Co-Authored-By: Claude Opus 5 <noreply@anthropic.com>

File: occlusion-sim/src/ubot/ubot_description/urdf/body/ubot_robot.urdf.xacro (robot description, xacro)
@@ -5,4 +5,5 @@
     <xacro:arg name="prefix" default=""/>
     <xacro:arg name="use_gazebo" default="false"/>
+    <xacro:arg name="sensor_profile" default="full"/>
     <xacro:include filename="$(find ubot_description)/urdf/body/ubot_base.urdf.xacro"/>
     <xacro:include filename="$(find ubot_description)/urdf/sensors/ubot_lidar.urdf.xacro"/>

File: occlusion-sim/src/ubot/ubot_description/urdf/gazebo/ubot_gazebo.urdf.xacro (robot description, xacro)
@@ -1,4 +1,20 @@
 <?xml version="1.0"?>
 <robot xmlns:xacro="http://www.ros.org/wiki/xacro">
+    <!--
+      Sensor cost profile. Rendering the depth camera and lidar dominates simulation speed:
+      in the full Sonoma Raceway world the 'full' profile runs at roughly RTF 0.2 on a
+      machine without GPU passthrough (/scan arrives at ~2 Hz instead of 10 Hz).
+        sensor_profile:=fast   half resolution, lower rates - use while developing/driving
+        sensor_profile:=full   nominal sensors - use for final captures
+      Pass it through the launch:  ros2 launch ubot_bringup sim.launch.py sensor_profile:=fast
+    -->
+    <xacro:arg name="sensor_profile" default="full"/>
+    <xacro:property name="profile" value="$(arg sensor_profile)"/>
+    <xacro:property name="lidar_samples"  value="${360 if profile == 'fast' else 720}"/>
+    <xacro:property name="lidar_rate"     value="${5 if profile == 'fast' else 10}"/>
+    <xacro:property name="camera_width"   value="${320 if profile == 'fast' else 640}"/>
+    <xacro:property name="camera_height"  value="${240 if profile == 'fast' else 480}"/>
+    <xacro:property name="camera_rate"    value="${10 if profile == 'fast' else 30}"/>
+    <xacro:property name="imu_rate"       value="${50 if profile == 'fast' else 100}"/>
     <xacro:macro name="ubot_gazebo" params="prefix">
         <gazebo>
@@ -19,5 +35,5 @@
             <sensor name="${prefix}lidar_sensor" type="gpu_lidar">
                 <topic>/scan</topic>
-                <update_rate>10</update_rate>
+                <update_rate>${lidar_rate}</update_rate>
                 <always_on>true</always_on>
                 <visualize>true</visualize>
@@ -25,5 +41,5 @@
                     <scan>
                         <horizontal>
-                            <samples>720</samples>
+                            <samples>${lidar_samples}</samples>
                             <resolution>1</resolution>
                             <min_angle>-3.14159</min_angle>
@@ -49,5 +65,5 @@
             <sensor name="${prefix}rgbd_camera" type="rgbd_camera">
                 <topic>${prefix}camera</topic>
-                <update_rate>30</update_rate>
+                <update_rate>${camera_rate}</update_rate>
                 <always_on>1</always_on>
                 <visualize>true</visualize>
@@ -55,6 +71,6 @@
                     <horizontal_fov>1.211</horizontal_fov>
                     <image>
-                        <width>640</width>
-                        <height>480</height>
+                        <width>${camera_width}</width>
+                        <height>${camera_height}</height>
                         <format>R8G8B8</format>
                     </image>
@@ -82,5 +98,5 @@
             <sensor name="${prefix}imu_sensor" type="imu">
                 <topic>/imu</topic>
-                <update_rate>100</update_rate>
+                <update_rate>${imu_rate}</update_rate>
                 <always_on>1</always_on>
                 <visualize>false</visualize>

Commit message: Add ubot_mono_nav: camera-only navigation, with the blind recoveries removed
The LiDAR-less stack (RGB -> metric depth -> /scan_mono -> nav2) existed only in a
local workspace copy and was in no branch here. Bring it in, plus the three URDF
changes it depends on, and fix three things that would have bitten on the robot.

Ported from the local copy (which predates the CAD body work, so this is a merge,
not a copy: taking it wholesale would have reverted the wheel friction fix and
replaced the OAK-D mesh with the old RealSense box):

  ubot_camera.urdf.xacro   `pitch` argument, POSITIVE = looking UP, applied on top
                           of the 4.09 deg down tilt the CamCase gives the OAK-D in
                           CAD, so net tilt = cad_tilt - pitch and pitch=0 is pure
                           CAD. The mesh visual origin is now computed symbolically
                           so it lands correctly at any tilt (checked at 0 and 0.13).
                           camera_rgb_frame and camera_optical_frame are now REAL
                           optical frames parented to camera_link; camera_depth_frame
                           stays body-aligned, as its use elsewhere assumes.
  ubot_gazebo.urdf.xacro   gz_frame_id -> camera_optical_frame, in both camera
  ubot_camera_gazebo       sensors. Gazebo publishes images and clouds in the optical
                           convention; stamping the body-aligned frame rotated every
                           projected point by 90 degrees, which looks plausible in
                           rviz and silently ruins depth_to_scan.
  ubot_robot.urdf.xacro    camera_pitch arg wired through to the camera macro.

Fixes, all three found by review rather than by running:

1. Recovery would have aborted navigation. behavior_plugins deliberately drops
   spin and backup (both move the robot through space a 65 deg camera cannot see),
   but nav2's DEFAULT behaviour trees still call Spin and BackUp, so the first
   recovery would hang on an action server that never appears. Ship trimmed trees
   in behavior_trees/ (clear the costmaps, then wait) and point bt_navigator at
   them from both launch files via RewrittenYaml.

2. Angular limits exceeded the hardware. max_vel_theta was 0.6 rad/s; in-place
   rotation actually saturates at ~0.3 because the tyres must scrub, and a stalled
   skid-steer makes odometry lie. Now 0.25, and the velocity smoother is capped to
   match with x min at 0.0 so nothing can emit a blind reverse.

3. The two stacks planned with different robot shapes. nav2_params_mono used
   robot_radius 0.15 while the lidar params use the measured 357 x 252 mm
   rectangle. Same footprint in both now, or the A/B comparison is not
   like-for-like.

Verified: the three packages build; scan_geometry --selftest passes 10/10;
check_urdf parses with use_gazebo true and false; camera_pitch 0 -> 4.09 deg down
and 0.13 -> 3.36 deg up; the installed trees call only loaded behaviours (Wait).
Not yet run on hardware.

Co-Authored-By: Claude Opus 5 <noreply@anthropic.com>

File: occlusion-sim/src/ubot/ubot_description/urdf/body/ubot_robot.urdf.xacro (robot description, xacro)
@@ -6,4 +6,8 @@
     <xacro:arg name="use_gazebo" default="false"/>
     <xacro:arg name="sensor_profile" default="full"/>
+    <!-- Camera tilt CORRECTION in radians, POSITIVE = looking UP, on top of the 4.09 deg
+         downward tilt the CamCase gives the OAK-D in CAD (confirmed against the robot:
+         lens centre 0.152 m off the floor). 0 unless the mount is physically bent. -->
+    <xacro:arg name="camera_pitch" default="0"/>
     <xacro:include filename="$(find ubot_description)/urdf/body/ubot_base.urdf.xacro"/>
     <xacro:include filename="$(find ubot_description)/urdf/sensors/ubot_lidar.urdf.xacro"/>
@@ -29,5 +33,6 @@
     prefix="$(arg prefix)" /> -->
     <xacro:ubot_camera
-    prefix="$(arg prefix)" />
+    prefix="$(arg prefix)"
+    pitch="$(arg camera_pitch)" />
     <xacro:ubot_rpi_camera
     prefix="$(arg prefix)" />

File: occlusion-sim/src/ubot/ubot_description/urdf/gazebo/ubot_camera_gazebo.urdf.xacro (robot description, xacro)
@@ -45,5 +45,9 @@
           <render_engine>ogre2</render_engine>
         </plugin>
-        <gz_frame_id>${prefix}camera_depth_frame</gz_frame_id>
+        <!-- Optical frame, not camera_depth_frame: Gazebo publishes images and
+                     clouds in the optical convention (Z forward), while camera_depth_frame
+                     is body-aligned. Stamping the body frame rotates every projected
+                     point by 90 degrees, which silently breaks depth_to_scan. -->
+                <gz_frame_id>${prefix}camera_optical_frame</gz_frame_id>
       </sensor>
     </gazebo>

File: occlusion-sim/src/ubot/ubot_description/urdf/gazebo/ubot_gazebo.urdf.xacro (robot description, xacro)
@@ -91,5 +91,9 @@
                     </depth_camera>
                 </camera>
-                <gz_frame_id>${prefix}camera_depth_frame</gz_frame_id>
+                <!-- Optical frame, not camera_depth_frame: Gazebo publishes images and
+                     clouds in the optical convention (Z forward), while camera_depth_frame
+                     is body-aligned. Stamping the body frame rotates every projected
+                     point by 90 degrees, which silently breaks depth_to_scan. -->
+                <gz_frame_id>${prefix}camera_optical_frame</gz_frame_id>
             </sensor>
         </gazebo>

File: occlusion-sim/src/ubot/ubot_description/urdf/sensors/ubot_camera.urdf.xacro (robot description, xacro)
@@ -4,6 +4,12 @@
     Luxonis OAK-D Lite depth camera in the front CamCase.
     camera_link sits at the centre of the RGB lens on the front face, X pointing out of
-    the lens. The CamCase tilts the camera 4.09 deg downward (camera_pitch).
-    Mesh: simplified 91 x 28 x 17.5 mm body with the three lenses, in Fusion world coords.
+    the lens. Mesh: simplified 91 x 28 x 17.5 mm body with the three lenses, exported in
+    Fusion world coordinates.
+    TILT. The CamCase pocket tilts the camera 4.09 deg (0.0714 rad) DOWN in CAD. The
+    `pitch` argument adds a correction measured on the real robot, POSITIVE = looking UP
+    (calibrate_pose.py measures it against the ground plane), so the net tilt is
+    cad_tilt - pitch and pitch=0 reproduces the CAD geometry exactly. Getting this wrong
+    puts every camera-derived obstacle at the wrong height, which is why depth_to_scan
+    reads the transform from TF rather than assuming it.
   -->
   <xacro:property name="camera_mass" value="0.061" />    <!-- OAK-D Lite datasheet -->
@@ -14,11 +20,18 @@
   <xacro:property name="camera_y" value="0.0" />
   <xacro:property name="camera_z" value="0.085654" />
-  <xacro:property name="camera_pitch" value="0.0714" />   <!-- rad, positive = looking down -->
-  <xacro:macro name="ubot_camera" params="prefix">
+  <xacro:property name="camera_cad_tilt" value="0.0714" />   <!-- rad, positive = looking down -->
+  <!-- Mesh position in the exported (Fusion world) frame; the visual origin below is the
+       inverse of the joint transform, computed symbolically because the tilt is variable. -->
+  <xacro:property name="camera_mesh_x" value="0.330149" />
+  <xacro:property name="camera_mesh_z" value="0.085654" />
+  <xacro:macro name="ubot_camera" params="prefix pitch:=0">
+    <!-- net tilt, positive = down -->
+    <xacro:property name="tilt" value="${camera_cad_tilt - pitch}" />
     <!--CAMERA_LINK (OAK-D Lite body)-->
     <link name="${prefix}camera_link">
       <visual>
         <!-- inverse of the joint transform, so the world-frame mesh lands in place -->
-        <origin xyz="-0.323197 0 -0.108988" rpy="0 ${-camera_pitch} 0"/>
+        <origin xyz="${-camera_mesh_x*cos(tilt) + camera_mesh_z*sin(tilt)} 0 ${-camera_mesh_x*sin(tilt) - camera_mesh_z*cos(tilt)}"
+                rpy="0 ${-tilt} 0"/>
         <geometry>
           <mesh filename="file://$(find ubot_description)/meshes/inspection/oakd_lite.stl" scale="0.001 0.001 0.001"/>
@@ -41,29 +54,38 @@
       <parent link="${prefix}base_link"/>
       <child link="${prefix}camera_link"/>
-      <origin xyz="${camera_x} ${camera_y} ${camera_z}" rpy="0 ${camera_pitch} 0"/>
+      <origin xyz="${camera_x} ${camera_y} ${camera_z}" rpy="0 ${tilt} 0"/>
     </joint>
-    <!-- CAMERA_DEPTH_FRAME (Optical frame for depth)
-         This follows ROS REP-103 conventions X is right, Y is down, Z is forward -->
+    <!-- WHICH FRAME IS WHICH, because getting this wrong rotates every
+         camera-derived obstacle by 90 degrees and still looks plausible:
+           camera_link           body frame:    X FORWARD, Y left, Z up
+           camera_depth_frame    body-aligned, identical to camera_link
+           camera_rgb_frame      OPTICAL:       X right, Y down, Z FORWARD
+           camera_optical_frame  OPTICAL, same as camera_rgb_frame
+         Images and point clouds use the OPTICAL convention, so anything that
+         projects pixels into 3D must be stamped camera_rgb_frame or
+         camera_optical_frame, never camera_depth_frame. -->
+    <!-- CAMERA_DEPTH_FRAME: kept for compatibility. NOT an optical frame
+         despite its old comment: it is aligned with camera_link. -->
     <link name="${prefix}camera_depth_frame"/>
     <joint name="${prefix}camera_depth_joint" type="fixed">
       <parent link="${prefix}camera_link"/>
       <child link="${prefix}camera_depth_frame"/>
-      <!-- Rotate to optical frame X right, Y down, Z forward -->
       <origin xyz="0 0 0" rpy="0 0 0"/>
     </joint>
-    <!-- CAMERA_RGB_FRAME (Optical frame for RGB) Typically aligned with depth frame-->
+    <!-- CAMERA_RGB_FRAME: the optical frame. X right, Y down, Z forward. -->
     <link name="${prefix}camera_rgb_frame"/>
     <joint name="${prefix}camera_rgb_joint" type="fixed">
       <parent link="${prefix}camera_link"/>
       <child link="${prefix}camera_rgb_frame"/>
-      <!-- Same orientation as depth frame -->
       <origin xyz="0 0 0" rpy="${-pi/2} 0 ${-pi/2}"/>
     </joint>
-    <!-- CAMERA_OPTICAL_FRAME (Alias for compatibility) -->
+    <!-- CAMERA_OPTICAL_FRAME: what Gazebo stamps its images and clouds with.
+         Was parented to camera_depth_frame with no rotation, which made it
+         body-aligned and its name a lie; it is now a real optical frame. -->
     <link name="${prefix}camera_optical_frame"/>
     <joint name="${prefix}camera_optical_joint" type="fixed">
-      <parent link="${prefix}camera_depth_frame"/>
+      <parent link="${prefix}camera_link"/>
       <child link="${prefix}camera_optical_frame"/>
-      <origin xyz="0 0 0" rpy="0 0 0"/>
+      <origin xyz="0 0 0" rpy="${-pi/2} 0 ${-pi/2}"/>
     </joint>
   </xacro:macro>
